File: kicad/PCA9685.sch (KiCad schematic (older format))
At the start: 28 parts, among them IC11 MAX3370, IC12 SN74LVC1G07, IC6 PCA9685, P1 CONN_3X16

Commit message: V1.0.5
Parts:
- JP3: symbol JUMPER3 -> JUMPER3-RESCUE-dronPi
Changed lines of the file:
@@
 $EndComp
 $Comp
-L JUMPER3 JP3
+L JUMPER3-RESCUE-dronPi JP3
 U 1 1 578EDC75
 P 7750 5550

Commit message: Add files via upload
Parts:
- IC12: value SN74LVC1G07 -> SN74AHC1G04
Changed lines of the file:
@@
 LIBS:contrib
 LIBS:valves
-LIBS:Raspberry_PI_B+
-LIBS:RPi_Hat-cache
-LIBS:mpu-9250
-LIBS:pixhawk2
-LIBS:PCA9685
-LIBS:microbuilder
-LIBS:pca9306
-LIBS:EMI
-LIBS:crystal
-LIBS:eelib
-LIBS:Carlolib-dev
-LIBS:NPN
-LIBS:DMMT5401
-LIBS:selfmade
-LIBS:3_16
 LIBS:dronPi-cache
-EELAYER 25 0
+EELAYER 26 0
 EELAYER END
 $Descr A4 11693 8268
@@
 $EndComp
 $Comp
-L GND #PWR021
+L GND-RESCUE-dronPi #PWR021
 U 1 1 5750EFE0
 P 9450 4850
+AR Path="/5750EFE0" Ref="#PWR021"  Part="1"
+AR Path="/574DDCCC/5750EFE0" Ref="#PWR021"  Part="1"
 F 0 "#PWR021" H 9450 4850 30  0001 C CNN
 F 1 "GND" H 9450 4780 30  0001 C CNN
@@
 $EndComp
 $Comp
-L GND #PWR022
+L GND-RESCUE-dronPi #PWR022
 U 1 1 5750F016
 P 4850 5400
+AR Path="/5750F016" Ref="#PWR022"  Part="1"
+AR Path="/574DDCCC/5750F016" Ref="#PWR022"  Part="1"
 F 0 "#PWR022" H 4850 5400 30  0001 C CNN
 F 1 "GND" H 4850 5330 30  0001 C CNN
@@
 P 8650 5900
 F 0 "IC12" H 8650 5431 45  0000 C CNN
-F 1 "SN74LVC1G07" H 8650 5347 45  0000 C CNN
+F 1 "SN74AHC1G04" H 8650 5347 45  0000 C CNN
 F 2 "Tinkerforge:SC70-5" H 8680 6050 20  0001 C CNN
 F 3 "" H 8650 5900 60  0001 C CNN
@@
 $EndComp
 $Comp
-L GND #PWR023
+L GND-RESCUE-dronPi #PWR023
 U 1 1 578EFE5A
 P 5800 6550
+AR Path="/578EFE5A" Ref="#PWR023"  Part="1"
+AR Path="/574DDCCC/578EFE5A" Ref="#PWR023"  Part="1"
 F 0 "#PWR023" H 5800 6550 30  0001 C CNN
 F 1 "GND" H 5800 6480 30  0001 C CNN
@@
 $EndComp
 $Comp
-L GND #PWR024
+L GND-RESCUE-dronPi #PWR024
 U 1 1 578F29AA
 P 9500 5900
+AR Path="/578F29AA" Ref="#PWR024"  Part="1"
+AR Path="/574DDCCC/578F29AA" Ref="#PWR024"  Part="1"
 F 0 "#PWR024" H 9500 5900 30  0001 C CNN
 F 1 "GND" H 9500 5830 30  0001 C CNN
@@
 +5v_SERV
 $Comp
-L GND #PWR025
+L GND-RESCUE-dronPi #PWR025
 U 1 1 578FACC1
 P 8050 6350
+AR Path="/578FACC1" Ref="#PWR025"  Part="1"
+AR Path="/574DDCCC/578FACC1" Ref="#PWR025"  Part="1"
 F 0 "#PWR025" H 8050 6350 30  0001 C CNN
 F 1 "GND" H 8050 6280 30  0001 C CNN
