File: kicad/fuente.sch (KiCad schematic (older format))
At the start: 30 parts, among them IC1 MIC5332, P2 PowerOff, Q1 MMBT3906LT1, Q2 DMG2305, U1 DMMT5401

Commit message: V1.0.5
Changed lines of the file:
@@
 P 6000 2300
 F 0 "D1" V 5900 2100 50  0000 L CNN
-F 1 "SMBJ5V" V 6050 1950 50  0000 L CNN
+F 1 "SMBJ5V" V 6150 2000 50  0000 L CNN
 F 2 "Tinkerforge:DO-214AA" H 6000 2300 50  0001 C CNN
 F 3 "" H 6000 2300 50  0000 C CNN
